File: solenoid_main_board/solenoid_main_board.kicad_sch (KiCad schematic)
At the start: 4 parts, among them J3 1x2 5.08, U1 solenoid_module, U2 Control_panel_module_comm, U4 MCU_module

Commit message: main board layout
Parts:
- J3: Mouser Part Number (none) -> 179-TB0012-508-02GR; Mouser number 179-TB0012-508-02GR -> (none)
Changed lines of the file:
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@@
 			)
 		)
-		(property "Mouser number" "179-TB0012-508-02GR"
+		(property "Mouser number" ""
 			(at 26.67 43.18 0)
 			(effects
@@
 			(effects
 				(font
+					(size 1.27 1.27)
+				)
+				(hide yes)
+			)
+		)
+		(property "Mouser Part Number" "179-TB0012-508-02GR"
+			(at 26.67 43.18 0)
+			(effects
+				(font
